Commit message: change each leg to 4 DOFs

File: urdf/crawler.xacro (robot description, xacro)
@@ -6,6 +6,8 @@
     <xacro:property name="M_body" value="5"/>
     <xacro:property name="R_up_leg" value="0.05"/>
-    <xacro:property name="L_up_leg" value="0.5"/>
-    <xacro:property name="M_up_leg" value="2"/>
+    <xacro:property name="L_up_leg" value="0.40"/>
+    <xacro:property name="L_up_con_leg" value="0.05"/>
+    <xacro:property name="M_up_leg" value="1.5"/>
+    <xacro:property name="M_up_con_leg" value="0.25"/>
     <xacro:property name="R_down_leg" value="0.025"/>
     <xacro:property name="L_down_leg" value="0.5"/>
@@ -19,4 +21,14 @@
     </xacro:macro>
     <xacro:macro name="joint2_property">
+        <axis xyz="0 0 1"/>
+        <dynamics damping="0.7" friction="0.0"/>
+        <limit effort="100.0" velocity="10.0" lower="0.0" upper="${pi*5/6}"/>
+    </xacro:macro>
+    <xacro:macro name="joint3_property">
+        <axis xyz="1 0 0"/>
+        <dynamics damping="0.7" friction="0.0"/>
+        <limit effort="100.0" velocity="10.0" lower="${-pi/2}" upper="${pi/2}"/>
+    </xacro:macro>
+    <xacro:macro name="joint4_property">
         <axis xyz="0 0 1"/>
         <dynamics damping="0.7" friction="0.0"/>

File: urdf/leg.xacro (robot description, xacro)
@@ -14,4 +14,42 @@
         </transmission>
         <link name="leg1_${suffix}">
+            <inertial>
+                <origin xyz="${L_up_con_leg/2} 0 0" rpy="0 ${pi/2} 0"/>
+                <mass value="${M_up_con_leg}" />
+                <inertia ixx="${M_up_con_leg * (1/12 * L_up_con_leg * L_up_con_leg + 1/4 * R_up_leg * R_up_leg)}" ixy="0" ixz="0" iyy="${M_up_con_leg * (1/12 * L_up_con_leg * L_up_con_leg + 1/4 * R_up_leg * R_up_leg)}" iyz="0" izz="${1/2 * M_up_con_leg * R_up_leg * R_up_leg}" />
+            </inertial>
+            <visual>
+                <origin xyz="${L_up_con_leg/2} 0 0" rpy="0 ${pi/2} 0"/>
+                <geometry>
+                    <cylinder length="${L_up_con_leg}" radius="${R_up_leg}"/>
+                </geometry>
+            </visual>
+            <collision>
+                <origin xyz="${L_up_con_leg/2} 0 0" rpy="0 ${pi/2} 0"/>
+                <geometry>
+                    <cylinder length="${L_up_con_leg}" radius="${R_up_leg}"/>
+                </geometry>
+            </collision>
+        </link>
+        <gazebo reference="leg1_${suffix}">
+            <material>Gazebo/Grey</material>
+        </gazebo>
+        <joint name="joint2_${suffix}" type="revolute">
+            <parent link="leg1_${suffix}"/>
+            <child link="leg2_${suffix}"/>
+            <origin xyz="${L_up_con_leg} 0 0" rpy="${-pi/2} 0 0"/>
+            <xacro:joint2_property/>
+        </joint>
+        <transmission name="tran2_${suffix}">
+            <type>transmission_interface/SimpleTransmission</type>
+            <joint name="joint2_${suffix}">
+                <hardwareInterface>hardware_interface/EffortJointInterface</hardwareInterface>
+            </joint>
+            <actuator name="act2_${suffix}">
+                <hardwareInterface>hardware_interface/EffortJointInterface</hardwareInterface>
+                <mechanicalReduction>1</mechanicalReduction>
+            </actuator>
+        </transmission>
+        <link name="leg2_${suffix}">
             <inertial>
                 <origin xyz="${L_up_leg/2} 0 0" rpy="0 ${pi/2} 0"/>
@@ -32,24 +70,62 @@
             </collision>
         </link>
-        <gazebo reference="leg1_${suffix}">
+        <gazebo reference="leg2_${suffix}">
             <material>Gazebo/Grey</material>
         </gazebo>
-        <joint name="joint2_${suffix}" type="revolute">
-            <parent link="leg1_${suffix}"/>
-            <child link="leg2_${suffix}"/>
-            <origin xyz="${L_up_leg} 0 0" rpy="${-pi/2} 0 0"/>
-            <xacro:joint2_property/>
+        <joint name="joint3_${suffix}" type="revolute">
+            <parent link="leg2_${suffix}"/>
+            <child link="leg3_${suffix}"/>
+            <origin xyz="${L_up_leg} 0 0" rpy="0 0 0"/>
+            <xacro:joint3_property/>
         </joint>
-        <transmission name="tran2_${suffix}">
+        <transmission name="tran3_${suffix}">
             <type>transmission_interface/SimpleTransmission</type>
-            <joint name="joint2_${suffix}">
+            <joint name="joint3_${suffix}">
                 <hardwareInterface>hardware_interface/EffortJointInterface</hardwareInterface>
             </joint>
-            <actuator name="act2_${suffix}">
+            <actuator name="act3_${suffix}">
                 <hardwareInterface>hardware_interface/EffortJointInterface</hardwareInterface>
                 <mechanicalReduction>1</mechanicalReduction>
             </actuator>
         </transmission>
-        <link name="leg2_${suffix}">
+        <link name="leg3_${suffix}">
+            <inertial>
+                <origin xyz="${L_up_con_leg/2} 0 0" rpy="0 ${pi/2} 0"/>
+                <mass value="${M_up_con_leg}" />
+                <inertia ixx="${M_up_con_leg * (1/12 * L_up_con_leg * L_up_con_leg + 1/4 * R_up_leg * R_up_leg)}" ixy="0" ixz="0" iyy="${M_up_con_leg * (1/12 * L_up_con_leg * L_up_con_leg + 1/4 * R_up_leg * R_up_leg)}" iyz="0" izz="${1/2 * M_up_con_leg * R_up_leg * R_up_leg}" />
+            </inertial>
+            <visual>
+                <origin xyz="${L_up_con_leg/2} 0 0" rpy="0 ${pi/2} 0"/>
+                <geometry>
+                    <cylinder length="${L_up_con_leg}" radius="${R_up_leg}"/>
+                </geometry>
+            </visual>
+            <collision>
+                <origin xyz="${L_up_con_leg/2} 0 0" rpy="0 ${pi/2} 0"/>
+                <geometry>
+                    <cylinder length="${L_up_con_leg}" radius="${R_up_leg}"/>
+                </geometry>
+            </collision>
+        </link>
+        <gazebo reference="leg3_${suffix}">
+            <material>Gazebo/Grey</material>
+        </gazebo>
+        <joint name="joint4_${suffix}" type="revolute">
+            <parent link="leg3_${suffix}"/>
+            <child link="leg4_${suffix}"/>
+            <origin xyz="${L_up_con_leg} 0 0" rpy="0 0 0"/>
+            <xacro:joint4_property/>
+        </joint>
+        <transmission name="tran4_${suffix}">
+            <type>transmission_interface/SimpleTransmission</type>
+            <joint name="joint4_${suffix}">
+                <hardwareInterface>hardware_interface/EffortJointInterface</hardwareInterface>
+            </joint>
+            <actuator name="act4_${suffix}">
+                <hardwareInterface>hardware_interface/EffortJointInterface</hardwareInterface>
+                <mechanicalReduction>1</mechanicalReduction>
+            </actuator>
+        </transmission>
+        <link name="leg4_${suffix}">
             <inertial>
                 <origin xyz="${L_down_leg/2} 0 0" rpy="0 ${pi/2} 0"/>
@@ -70,9 +146,9 @@
             </collision>
         </link>
-        <gazebo reference="leg2_${suffix}">
+        <gazebo reference="leg4_${suffix}">
             <material>Gazebo/Orange</material>
         </gazebo>
         <joint name="end_joint_${suffix}" type="fixed">
-            <parent link="leg2_${suffix}"/>
+            <parent link="leg4_${suffix}"/>
             <child link="foot_${suffix}"/>
             <origin xyz="${L_down_leg + R_foot} 0 0" rpy="0 0 0"/>

Commit message: speedup simulation and fix warning

File: urdf/crawler.xacro (robot description, xacro)
@@ -37,4 +37,9 @@
     <xacro:include filename="$(find crawler)/urdf/leg.xacro" />
     <xacro:include filename="$(find crawler)/urdf/crawler.gazebo" />
+    <link name="dummy"/>
+    <joint name="dummy_joint" type="fixed">
+        <parent link="dummy"/>
+        <child link="base"/>
+    </joint>
     <link name="base">
         <inertial>

Commit message: Add walkEnv, modify robot joint limit and initial pose

File: urdf/crawler.xacro (robot description, xacro)
@@ -18,10 +18,10 @@
         <axis xyz="0 0 1"/>
         <dynamics damping="0.7" friction="0.0"/>
-        <limit effort="100.0" velocity="10.0" lower="${-pi/2}" upper="${pi/2}"/>
+        <limit effort="100.0" velocity="10.0" lower="${-pi/4}" upper="${pi/4}"/>
     </xacro:macro>
     <xacro:macro name="joint2_property">
         <axis xyz="0 0 1"/>
         <dynamics damping="0.7" friction="0.0"/>
-        <limit effort="100.0" velocity="10.0" lower="0.0" upper="${pi*5/6}"/>
+        <limit effort="100.0" velocity="10.0" lower="${-pi/4}" upper="${pi/4}"/>
     </xacro:macro>
     <xacro:macro name="joint3_property">
@@ -33,5 +33,36 @@
         <axis xyz="0 0 1"/>
         <dynamics damping="0.7" friction="0.0"/>
-        <limit effort="100.0" velocity="10.0" lower="0.0" upper="${pi*5/6}"/>
+        <limit effort="100.0" velocity="10.0" lower="${-pi/3}" upper="${pi/3}"/>
+    </xacro:macro>
+    <xacro:macro name="leg_friction_property">
+        <collision>
+            <surface>
+                <friction>
+                    <ode>
+                        <mu>10</mu>
+                        <mu2>10</mu2>
+                    </ode>
+                </friction>
+            </surface>
+        </collision>
+    </xacro:macro>
+    <xacro:macro name="foot_property">
+        <collision>
+            <surface>
+                <contact>
+                    <ode>
+                        <kp>5e8</kp>
+                        <kd>0.5</kd>
+                        <min_depth>0.01</min_depth>
+                    </ode>
+                </contact>
+                <friction>
+                    <ode>
+                        <mu>10</mu>
+                        <mu2>10</mu2>
+                    </ode>
+                </friction>
+            </surface>
+        </collision>
     </xacro:macro>
     <xacro:include filename="$(find crawler)/urdf/leg.xacro" />

File: urdf/leg.xacro (robot description, xacro)
@@ -33,4 +33,5 @@
         </link>
         <gazebo reference="leg1_${suffix}">
+            <xacro:leg_friction_property/>
             <material>Gazebo/Grey</material>
         </gazebo>
@@ -38,5 +39,5 @@
             <parent link="leg1_${suffix}"/>
             <child link="leg2_${suffix}"/>
-            <origin xyz="${L_up_con_leg} 0 0" rpy="${-pi/2} 0 0"/>
+            <origin xyz="${L_up_con_leg} 0 0" rpy="${-pi/2} ${pi/8} 0"/>
             <xacro:joint2_property/>
         </joint>
@@ -71,4 +72,5 @@
         </link>
         <gazebo reference="leg2_${suffix}">
+            <xacro:leg_friction_property/>
             <material>Gazebo/Grey</material>
         </gazebo>
@@ -109,4 +111,5 @@
         </link>
         <gazebo reference="leg3_${suffix}">
+            <xacro:leg_friction_property/>
             <material>Gazebo/Grey</material>
         </gazebo>
@@ -114,5 +117,5 @@
             <parent link="leg3_${suffix}"/>
             <child link="leg4_${suffix}"/>
-            <origin xyz="${L_up_con_leg} 0 0" rpy="0 0 0"/>
+            <origin xyz="${L_up_con_leg} 0 0" rpy="0 0 ${pi/3}"/>
             <xacro:joint4_property/>
         </joint>
@@ -147,4 +150,5 @@
         </link>
         <gazebo reference="leg4_${suffix}">
+            <xacro:leg_friction_property/>
             <material>Gazebo/Orange</material>
         </gazebo>
@@ -174,15 +178,5 @@
         </link>
         <gazebo reference="foot_${suffix}">
-            <collision>
-                <surface>
-                    <contact>
-                        <ode>
-                            <kp>5e8</kp>
-                            <kd>0.5</kd>
-                            <min_depth>0.01</min_depth>
-                        </ode>
-                    </contact>
-                </surface>
-            </collision>
+            <xacro:foot_property/>
             <material>Gazebo/Black</material>
         </gazebo>
